File: Orp-pH Board/Orp-pH Board.kicad_sch (KiCad schematic)
At the start: 47 parts, among them J1 Conn_Coaxial, J2 Conn_Coaxial, J3 Conn_01x04_Male, U1 LMP7721MA/NOPB, U2 LMP7721MA/NOPB, U3 ADS1115IDGS, U4 ADM3260

Commit message: fixed small errors on the schema
Parts:
- TP3: value TestPoint Vcc -> TestPoint GND
Connections:
- net GNDin: no longer names the net of C12.2, C13.2, J3.1 (Pin_1), R23.1, R24.1, U4.4 (VDDP), U4.9 (VIN)
Changed lines of the file:
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@@
   (junction (at 243.205 106.68) (diameter 0) (color 0 0 0 0)
-  )
-  (junction (at 257.81 118.745) (diameter 0) (color 0 0 0 0)
   )
   (junction (at 138.43 121.92) (diameter 0) (color 0 0 0 0)
@@
     (stroke (width 0) (type default) (color 0 0 0 0))
   )
-  (wire (pts (xy 257.81 118.745) (xy 257.81 138.43))
+  (wire (pts (xy 257.81 114.3) (xy 257.81 138.43))
     (stroke (width 0) (type default) (color 0 0 0 0))
   )
@@
     (stroke (width 0) (type default) (color 0 0 0 0))
   )
-  (wire (pts (xy 255.27 118.745) (xy 257.81 118.745))
-    (stroke (width 0) (type default) (color 0 0 0 0))
-  )
   (wire (pts (xy 175.26 105.41) (xy 175.26 107.95))
     (stroke (width 0) (type default) (color 0 0 0 0))
@@
   )
   (wire (pts (xy 83.82 73.66) (xy 83.82 77.47))
-    (stroke (width 0) (type default) (color 0 0 0 0))
-  )
-  (wire (pts (xy 257.81 114.3) (xy 257.81 118.745))
     (stroke (width 0) (type default) (color 0 0 0 0))
   )
@@
     (effects (font (size 1.27 1.27)) (justify right))
     (property "Intersheet References" "${INTERSHEET_REFS}" (id 0) (at 156.3369 157.4006 0)
-      (effects (font (size 1.27 1.27)) (justify right) hide)
-    )
-  )
-  (global_label "GNDin" (shape bidirectional) (at 255.27 118.745 180) (fields_autoplaced)
-    (effects (font (size 1.27 1.27)) (justify right))
-    (property "Intersheet References" "${INTERSHEET_REFS}" (id 0) (at 247.2326 118.6656 0)
       (effects (font (size 1.27 1.27)) (justify right) hide)
     )
@@
       (effects (font (size 1.27 1.27)) (justify left))
     )
-    (property "Value" "TestPoint Vcc" (id 1) (at 245.11 91.3129 0)
+    (property "Value" "TestPoint GND" (id 1) (at 245.11 91.3129 0)
       (effects (font (size 1.27 1.27)) (justify left))
     )
@@
     )
     (path "/5f17c5ec-8737-42e1-8af1-ed7be1511e43"
-      (reference "TP3") (unit 1) (value "TestPoint Vcc") (footprint "TestPoint:TestPoint_Pad_D2.0mm")
+      (reference "TP3") (unit 1) (value "TestPoint GND") (footprint "TestPoint:TestPoint_Pad_D2.0mm")
     )
     (path "/483efb2f-3e22-4b2a-8c32-eb5e111155a9"

Commit message: fixed gain error in label of schematics
Other:
- note added: "pH gain: 7.62 range: +/- 2048mV over 2.5V mid range range pH: from 2.37 to 11.63 Orp gain: 2.32 range Orp: +/- 1077mV"
- note removed: "pH gain: 6.62 range: +/- 2048mV over 2.5V mid range range pH: from 2.37 to 11.63 Orp gain: 2.32 range Orp: +/- 1077mV"
Changed lines of the file:
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@@
     (effects (font (size 3 3)) (justify left bottom))
   )
-  (text "pH\ngain: 6.62\nrange: +/- 2048mV over 2.5V mid range\nrange pH: from 2.37 to 11.63\n\nOrp\ngain: 2.32\nrange Orp: +/- 1077mV"
+  (text "pH\ngain: 7.62\nrange: +/- 2048mV over 2.5V mid range\nrange pH: from 2.37 to 11.63\n\nOrp\ngain: 2.32\nrange Orp: +/- 1077mV"
     (at 179.07 58.42 0)
     (effects (font (size 3 3)) (justify left bottom))
